File: KiKad/USBBattPack3.3VoltageRegulator.kicad_sch (KiCad schematic)
At the start: 2 parts, among them U10 MCP1825S, U11 MCP1826S

Commit message: some work
Parts:
- added C301, C303: 100n, symbol Device:C
- added C302: 10u, symbol Device:C
- added C304, C305: 22u, symbol Device:C
- added C306: 75p, symbol Device:C
- added C307, C309: 2u2, Capacitor_SMD:C_0805_2012Metric, symbol Device:C
- added C308: Cx, Capacitor_SMD:C_0805_2012Metric, symbol Device:C
- added L301: 100-600R, Inductor_SMD:L_0805_2012Metric, symbol Device:L_Ferrite_Small
- added L302: 15u, symbol Device:L_Iron_Small
- added R301, R302: DNP, symbol Device:R
- added R303: 100k, symbol Device:R
- added R304: 13k3, symbol Device:R
- added R305: Rx, Resistor_SMD:R_0805_2012Metric, symbol Device:R
- added R306: x, symbol Device:R
- added U302: TPS54202DDC, Package_TO_SOT_SMD:SOT-23-6, symbol Regulator_Switching:TPS54202DDC
Connections:
- new net: C303.1, U302.6 (BOOT)
- new net: C303.2, L302.1, U302.2 (SW)
- new net: C304.1, C305.1, C306.1, L302.2, R303.1
- new net: C301.1, C302.1, C308.1, C309.1, L301.2, R301.1, U302.3 (VIN)
- new net: C308.2, R305.2
- new net: R301.2, R302.1, U302.5 (EN)
- new net: C306.2, R303.2, R304.1, U302.4 (FB)
- new net: R304.2, R306.1
- new net GND: C301.2, C302.2, C304.2, C305.2, C307.2, C309.2, R302.2, R305.1, R306.2, U302.1 (GND)
- new net VDD: C307.1, L301.1
Other:
- note added: "5V: 75pF 3.3V: 56pF"
- note added: "Cout, for example: GRM32ER71E226KE15"
- note added: "EN float to enable"
- note added: "F=500kHz(390-630kHz) Also: TPS56200"
- note added: "MCP1825S Imax: 0.5A Vdropout: 210mB(typ), 350mV(max) MCP1826S Imax: 1A Vdropout: 250mB(typ), 400mV(max)"
- note added: "Vin: 4.5V-28V Imax: 2A"
- note added: "Vout = 0.596*(Rt/Rb+1) 5V: 100k / 13.3k 5.44V: 100k / 12.3k"
- moved on the sheet: U10, U11
