File: KiKad/USB PD.kicad_sch (KiCad schematic)
At the start: 6 parts, among them J101 Conn_02x07_Odd_Even, J4 USB_C_Receptacle_PowerOnly_6P, J5 USB_C_Receptacle_USB2.0_14P, U2 INA181, U3 INA219AxDCN

Commit message: some work
Parts:
- removed R101: R, symbol Device:R
- removed U2: INA181, Package_TO_SOT_SMD:SOT-23-6, symbol Amplifier_Current:INA181
- removed U3: INA219AxDCN, Package_TO_SOT_SMD:SOT-23-8, symbol Sensor_Energy:INA219AxDCN
- added Q301: Si2369, symbol Device:Q_PMOS_GSD
- added Q302: Si2338, symbol Device:Q_NMOS_GSD
- added R320: 100k, symbol Device:R
- added R321: 300k, symbol Device:R
- J101: value Conn_02x07_Odd_Even -> POWER_OUT
Connections:
- net GND: now also J101.10 (Pin_10), J101.12 (Pin_12), J101.14 (Pin_14), J101.2 (Pin_2), J101.4 (Pin_4), J101.6 (Pin_6), J101.8 (Pin_8), Q302.2 (S), R321.2
- net +BATT: now reaches J101.11 (Pin_11)
- net VBUS: now reaches J101.13 (Pin_13)
- net POWER_5V_ENABLE: now reaches J101.9 (Pin_9)
- net POWER_5V_ENABLE: now also Q302.1 (G), R321.1
- new net: Q301.1 (G), Q302.3 (D), R320.2
- new net 3.3V Voltage Regulator1/VDD: Q301.2 (S), R320.1
- new net 5V Voltage Regulator/VDD: Q301.3 (D)
Other:
- sheet 3.3V Voltage Regulator renamed 5V Voltage Regulator
- sheet Host Cotroller renamed Host Controller
- added sheet 3.3V Voltage Regulator1 (USBBattPack33VoltageRegulator.kicad_sch)
- sheet 5V Voltage Regulator: file USBBattPack3.3VoltageRegulator.kicad_sch -> USBBattPack5VoltageRegulator.kicad_sch
- sheet 5V Voltage Regulator ports: added +3.3VA, +5V, 5V_SENSE_I, 5V_SENSE_V, GND, GNDA, VDD, V_REF; removed none
- sheet Host Controller ports: added +3.3VA, GND, GNDA, SENSE_I1, SENSE_I2, SENSE_I3, SENSE_I4, SENSE_V1, SENSE_V2, SENSE_V3, SENSE_V4, VDD, V_REF; removed none
- moved on the sheet: J101

Commit message: some work
Parts:
- added C101: 4n7, Capacitor_SMD:C_0805_2012Metric, symbol Device:C
- added JP101: SysPower, symbol Jumper:Jumper_3_Bridged12
- renumbered J4 to J101, J5 to J102, J101 to J103, Q302 to Q101, Q301 to Q102, R320 to R101, R321 to R102
Connections:
- net +BATT: now also JP101.3 (B)
- net 3.3V Voltage Regulator1/VDD: now also JP101.2 (C)
- net Charger/CC1: now also J101.A5 (CC1), J102.A5 (CC1)
- net Charger/CC2: now also J101.B5 (CC2), J102.B5 (CC2)
- net Charger/D+: now also J102.A6 (D+), J102.B6 (D+)
- net Charger/D-: now also J102.A7 (D-), J102.B7 (D-)
- net GND: now also J101.A12 (GND), J101.B12 (GND), J102.A1 (GND), J102.A12 (GND), J102.B1 (GND), J102.B12 (GND), C101.2
- net VBUS: now also J101.A9 (VBUS), J101.B9 (VBUS), J102.A4 (VBUS), J102.A9 (VBUS), J102.B4 (VBUS), J102.B9 (VBUS)
- net at J102.S1 (SHIELD): now also J101.S1 (SHIELD), C101.1
- new net Charger/VSYS: JP101.1 (A)
Other:
- sheet 3.3V Voltage Regulator1 ports: added +3.3VA, 3.3V_SENSE_I, 3.3V_SENSE_U, GNDA, V_REF; removed none
- sheet 5V Voltage Regulator ports: added 5V_SENSE_U; removed 5V_SENSE_V
- sheet Battery Pack ports: added +3.3VA, BATT_SENSE_I, BATT_SENSE_U, GNDA, V_REF; removed none
- sheet Host Controller ports: added CHARGER_CE, CHARGER_INT, CHARGER_QON, STUSB_ALERT; removed none
- moved on the sheet: J101, J102, J103, Q101, Q102, R101, R102
