File: KiKad/USBBattPack33VoltageRegulator.kicad_sch (KiCad schematic)
At the start: 36 parts, among them U303 TPS54202DDC, U304 MCP1826S

Commit message: some work
Parts:
- removed C315, C320: 100n, symbol Device:C
- removed C316, C318, C324, C326: 2u2, Capacitor_SMD:C_0805_2012Metric, symbol Device:C
- removed C317, C325: Cx, Capacitor_SMD:C_0805_2012Metric, symbol Device:C
- removed C319: 10u, symbol Device:C
- removed C321, C322: 22u, symbol Device:C
- removed C323: 75p, symbol Device:C
- removed C327: 4.7u, Capacitor_SMD:C_0805_2012Metric, symbol Device:C
- removed C328: 1u, Capacitor_SMD:C_0805_2012Metric, symbol Device:C
- removed L304, L306: 100-600R, Inductor_SMD:L_0805_2012Metric, symbol Device:L_Ferrite_Small
- removed L305: 15u, symbol Device:L_Iron_Small
- removed R308, R311: DNP, symbol Device:R
- removed R309: 100k, symbol Device:R
- removed R310, R312: Rx, Resistor_SMD:R_0805_2012Metric, symbol Device:R
- removed R313: 13k3, symbol Device:R
- removed R314: x, symbol Device:R
- removed TP311, TP316: in, symbol Connector:TestPoint
- removed TP312, TP317: dc-in-f, symbol Connector:TestPoint
- removed TP313, TP318: dc-out, symbol Connector:TestPoint
- removed TP314, TP319: dc-out-f, symbol Connector:TestPoint
- removed TP315, TP320: out, symbol Connector:TestPoint
- removed U303: TPS54202DDC, Package_TO_SOT_SMD:SOT-23-6, symbol Regulator_Switching:TPS54202DDC
- removed U304: MCP1826S, symbol Regulator_Linear:MCP1826S
- added C601, C603, C610, C612: 2u2, Capacitor_SMD:C_0805_2012Metric, symbol Device:C
- added C602, C611: Cx, Capacitor_SMD:C_0805_2012Metric, symbol Device:C
- added C604: 10u, symbol Device:C
- added C605, C606, C614: 100n, symbol Device:C
- added C607, C608: 22u, symbol Device:C
- added C609: 56p, symbol Device:C
- added C613: 4.7u, Capacitor_SMD:C_0805_2012Metric, symbol Device:C
- added C615: 1u, Capacitor_SMD:C_0805_2012Metric, symbol Device:C
- added JP601: Ref, symbol Jumper:Jumper_3_Bridged12
- added L601, L603: 100-600R, Inductor_SMD:L_0805_2012Metric, symbol Device:L_Ferrite_Small
- added L602: 10u, symbol Device:L_Iron_Small
- added R601, R607: Rx, Resistor_SMD:R_0805_2012Metric, symbol Device:R
- added R602, R603: DNP, symbol Device:R
- added R604: 100k, symbol Device:R
- added R605: 18k9, symbol Device:R
- added R606: x, symbol Device:R
- added R608: 16.5m, symbol Device:R
- added TP601, TP602: in, symbol Connector:TestPoint
- added TP603, TP604: dc-in-f, symbol Connector:TestPoint
- added TP605, TP606: dc-out, symbol Connector:TestPoint
- added TP607, TP608: dc-out-f, symbol Connector:TestPoint
- added TP609, TP610: out, symbol Connector:TestPoint
- added U601: TPS54202DDC, Package_TO_SOT_SMD:SOT-23-6, symbol Regulator_Switching:TPS54202DDC
- added U602: MCP1826S-3.3, symbol Regulator_Linear:MCP1826S
- added U603: INA214, symbol myLib:INA21x
Connections:
- net +3.3V: now also R608.2, U603.5 (-)
- net GND: now also C601.2, C603.2, C604.2, C605.2, C607.2, C608.2, C610.2, C612.2, C613.2, C615.2, R601.1, R603.2, R606.2, R607.1, TP601.1, TP603.1, TP605.1, TP607.1, TP609.1, U601.1 (GND), U602.2 (GND)
- net VDD: now also C601.1, L601.1, TP602.1
- new net: C602.2, R601.2
- new net: C615.1, R608.1, TP610.1, U602.3 (VO), U603.4 (+)
- new net: C609.2, R604.2, R605.1, U601.4 (FB)
- new net: R605.2, R606.1
- new net: R602.2, R603.1, U601.5 (EN)
- new net: C611.2, R607.2
- new net: C606.2, L602.1, U601.2 (SW)
- new net: C606.1, U601.6 (BOOT)
- new net: JP601.2 (C), U603.1 (Ref)
- new net +3.3VA: C614.1, U603.3 (V+)
- new net 3.3V_SENSE_I: U603.6 (Out)
- new net DC3.3_INPUT: C602.1, C603.1, C604.1, C605.1, L601.2, R602.1, TP604.1, U601.3 (VIN)
- new net DC3.3_OUT: C607.1, C608.1, C609.1, C610.1, L602.2, L603.1, R604.1, TP606.1
- new net DC3.3_OUT_F: C611.1, C612.1, C613.1, L603.2, TP608.1, U602.1 (VI)
- new net GNDA: C614.2, JP601.1 (A), U603.2 (GND)
- new net V_REF: JP601.3 (B)
Other:
- note added: "F=500kHz(390-630kHz) Also: TPS56220x"
- note added: "INA21x Vadc(max) - 3.3V Isense(max) - 1A Vsense(max) - 10mV ----------------------- Gain=500 (INA211): Vsense = 3.3V/500 = 6.6mV Rsense = 6.6mOgm Gain=200 (INA210): Vsense = 3.3V/200 = 16.5mV Rsense = 16.5mOgm Gain=100 (INA214): Vsense = 3.3V/100 = 33mV Rsense = 33mOgm"
- note added: "Rb=Rt*0.586/(Vout-0.596) Vout = 0.596*(Rt/Rb+1) 3.3V: 100k / 22.1k 3.75V: 100k / 18.9k"
- note removed: "F=500kHz(390-630kHz) Also: TPS56200"
- note removed: "Vout = 0.596*(Rt/Rb+1) 5V: 100k / 13.3k 5.44V: 100k / 12.3k"
