File: KiKad/USBBattPack5VoltageRegulator.kicad_sch (KiCad schematic)
At the start: 40 parts, among them U11 MCP1826S-5.0, U302 TPS54202DDC, U308 INA214

Commit message: some work
Parts:
- JP501: renamed from JP301; value Jumper_3_Bridged12 -> Ref
- gave numbers to parts that had none: 1
- renumbered C307 to C501, C308 to C502, C309 to C503, C302 to C504, C301 to C505, C303 to C506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
