File: KiKad/USBBattPackCharger.kicad_sch (KiCad schematic)
At the start: 60 parts, among them J2 BATT_NTC, Q1 PMOS, Q2 PMOS, SW1 BQ_RESET, SW2 STUSB_RESET, U6 STUSB4500QTR, U7 BQ25792

Commit message: some work
Parts:
- added C224: 100n, symbol Device:C
- added R220: 30m, symbol Device:R
- added U203: INA213, symbol myLib:INA21x
- C201: renamed from C20; footprint (none) -> Capacitor_SMD:C_0805_2012Metric
- renumbered C4 to C202, C23 to C203, C2 to C204, C22 to C205, C3 to C206, C1 to C207, C19 to C208, C21 to C209, C10 to C210, C9 to C211, C8 to C212, C13 to C213, C11 to C214, C5 to C215, C12 to C216, C6 to C217, C14 to C218, C7 to C219, C15 to C220, C16 to C221, C17 to C222, C18 to C223, D3 to D201, D4 to D202, D2 to D203, D5 to D204, D7 to D205, D8 to D206, D6 to D207, D1 to D208, J2 to J201, JP1 to JP201, L1 to L201, Q1 to Q201, Q2 to Q202, R11 to R201, R19 to R202, R9 to R203, R13 to R204, R2 to R205, R10 to R206, R15 to R207, R16 to R208, R5 to R209, R6 to R210, R17 to R211, R12 to R212, R7 to R213, R8 to R214, R18 to R215, R3 to R216, R4 to R217, R14 to R218, R1 to R219, SW2 to SW201, SW1 to SW202, TP1 to TP201, U6 to U201, U7 to U202
Connections:
- new net +3.3VA: C224.1, U203.3 (V+)
- new net BATT_SENSE_I: U203.6 (Out)
- new net GNDA: C224.2, U203.2 (GND)
Other:
- moved on the sheet: C218
