File: KiKad/batteryPack.kicad_sch (KiCad schematic)
At the start: 66 parts, among them J3 BATT_NTP, Q3 N-MOSFET, Q4 N-MOSFET, Q5 N-MOSFET, Q6 N-MOSFET, Q7 N-MOSFET, Q8 N-MOSFET, Q9 PMOS, U9 BQ25792

Commit message: some work
Parts:
- added C306: 100n, symbol Device:C
- added R310: 30m, symbol Device:R
- added SW301: BattSwitch, symbol Switch:SW_SPDT
- added TP306: Sense+, symbol Connector:TestPoint
- added TP307: Sense-, symbol Connector:TestPoint
- added U301: INA213, symbol myLib:INA21x
- BT301: renamed from BT4; footprint (none) -> Battery:BatteryHolder_Keystone_1042_1x18650
- BT302: renamed from BT3; footprint (none) -> Battery:BatteryHolder_Keystone_1042_1x18650
- BT303: renamed from BT2; footprint (none) -> Battery:BatteryHolder_Keystone_1042_1x18650
- BT304: renamed from BT1; footprint (none) -> Battery:BatteryHolder_Keystone_1042_1x18650
- R312: renamed from R30; value RSNS -> 30m
- U302: renamed from U9; value BQ25792 -> BQ77915
- renumbered C26 to C301, C29 to C302, C28 to C303, C27 to C304, C30 to C305, C32 to C307, C31 to C308, C33 to C309, C24 to C310, C25 to C311, D11 to D301, D10 to D302, D9 to D303, J3 to J301, JP3 to JP301, JP2 to JP302, Q3 to Q301, Q6 to Q302, Q5 to Q303, Q4 to Q304, Q7 to Q305, Q9 to Q306, Q8 to Q307, R21 to R301, R27 to R302, R25 to R303, R23 to R304, R22 to R305, R28 to R306, R26 to R307, R24 to R308, R29 to R309, R36 to R311, R37 to R313, R38 to R314, R35 to R315, R20 to R316, R40 to R317, R41 to R318, R33 to R319, R42 to R320, R31 to R321, R32 to R322, R34 to R323, TP2 to TP301, TP3 to TP302, TP4 to TP303, TP5 to TP304, TP6 to TP305, TP17 to TP308, TP10 to TP309, TP16 to TP310, TP11 to TP311, TP15 to TP312, TP14 to TP313, TP13 to TP314, TP12 to TP315, TP7 to TP316, TP8 to TP317, TP9 to TP318
Connections:
- net +BATT: now also SW301.1 (A)
- net GND: now also R310.1; no longer R312.1
- net at C307.2, C308.2, R311.2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: now also TP306.1
- net at C308.1, C309.1, R313.2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: now also TP307.1
- net at Q305.3 (S), R312.2, R313.1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: now also U301.5 (-)
- new net: R310.2, R312.1, U301.4 (+)
- new net +3.3VA: C306.1, U301.3 (V+)
- new net BATT+: SW301.2 (B)
- new net BATT_SENSE_I: U301.6 (Out)
- new net GNDA: C306.2, U301.2 (GND)
- new net V_REF: U301.1 (Ref)
Other:
- note added: "INA21x Vadc(max) - 3.3V / 2 = 1.65V (bidirectional) Isense(max) - 1A ----------------------- Gain=50 (INA213): Rsense - 60mV Vsense = 1A * 60mR * 50 = 3V Gain=50 (INA213): Rsense - 30mV Vsense = 1A * 30mR * 50 = 1.5V"
